File: sipariş/ATESLEME.brd (EAGLE design)
At the start: 34.6 x 56.6 mm, 54 parts, among them U1 ADXL345PATRICK, U3 AMS1117-3.3

Commit message: LOGO was uploaded
Parts:
- moved VDD1 0.25 mm to (26.8, 35.9)
- moved VDD2 0.25 mm to (13.9, 35.1)
Routing:
- net 3.3V: track 138.2 -> 138.7 mm
