File: STM32F103C8T6/ATESLEME.sch (EAGLE design)
At the start: 54 parts, among them U1 ADXL345PATRICK, U7 AMS1117-3.3

Commit message: New version of boards with new controller was designed
Parts:
- removed OSC: (no value), ABMM2-8.000MHZ-E2-T:ABMM2-8.000MHZ-E2-T
- removed U7: AMS1117-3.3, AMS1117-3.3:AMS1117-3.3
- added NRST: 10k, SparkFun-Resistors:2.0KOHM1/10W5%(0603)
- added U3: AMS1117-3.3, AMS1117-3.3:AMS1117-3.3
- added Y2: ABM2B-8.000MHZ-10-1-U-T, ABM3B-26.000MHZ-10-1-U-T:ABM3B-26.000MHZ-10-1-U-T
Connections:
- new net HT: U3.HT
- new net IN1: U1.INT1, U2A.PB9
- new net IN2: U1.INT2, U2A.PB8
- new net INT1: LPS-1.INT1, U2A.PB5
- net 3.3V: now also NRST.2
- net GND: now also U3.ADJ, Y2.GND; no longer U7.ADJ/GND
- net N$1: now also U3.VOUT; no longer U7.VOUT
- net NRST: now also NRST.1
- net OSC_OUT: now also Y2.3; no longer OSC.OUT
- net OSC_ıN: now also Y2.1; no longer OSC.IN
- net VNR: now also U3.VIN; no longer U7.VIN
Other:
- note added: "APOGEE"
- note added: "MAIN"
- note removed: "APOGEE and MAIN"
- note removed: "İŞARETÇİLER"
- moved on the sheet: CRST, L1, OSCC1, OSCC2, SCL_3V3, SDA_3V3, VBAT, VDD, VDD1, VDD2, VDD3, VDDA1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
