File: STM32F102CBT6/ATESLEME.sch (EAGLE design)
At the start: 55 parts, among them U1 ADXL345PATRICK, U3 AMS1117-3.3, U4 STM32F102CBT6, Y2 ABM2B-8.000MHZ-10-1-U-T

Commit message: packages was modified according to stock situation
Parts:
- G1, G2: value 20 -> 22
- L1: value BLM15HB221SN1 -> (none); device inductors:BLM15HB221SN1 -> 52101-101-REV-A_v16:RC-MASTER-SMD_FB_0805MP
Changed lines of the file:
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@@
 <part name="VBAT_D" library="SparkFun-Resistors" deviceset="2.0KOHM1/10W5%(0603)" device="" value="3.3k"/>
 <part name="GND24" library="SparkFun" deviceset="GND" device=""/>
-<part name="G1" library="SparkFun-Resistors" deviceset="2.0KOHM1/10W5%(0603)" device="" value="20"/>
+<part name="G1" library="SparkFun-Resistors" deviceset="2.0KOHM1/10W5%(0603)" device="" value="22"/>
 <part name="U8" library="IRLML6344TRPBF" deviceset="IRLML6344TRPBF" device=""/>
 <part name="GND30" library="SparkFun-PowerSymbols" library_urn="urn:adsk.eagle:library:530" deviceset="GND" device=""/>
 <part name="S" library="SparkFun-Resistors" deviceset="2.0KOHM1/10W5%(0603)" device="" value="3.3k"/>
-<part name="G2" library="SparkFun-Resistors" deviceset="2.0KOHM1/10W5%(0603)" device="" value="20"/>
+<part name="G2" library="SparkFun-Resistors" deviceset="2.0KOHM1/10W5%(0603)" device="" value="22"/>
 <part name="U9" library="IRLML6344TRPBF" deviceset="IRLML6344TRPBF" device=""/>
 <part name="GND31" library="SparkFun-PowerSymbols" library_urn="urn:adsk.eagle:library:530" deviceset="GND" device=""/>
@@
 <part name="ADXLC1" library="SparkFun-Capacitors" library_urn="urn:adsk.eagle:library:510" deviceset="0.1UF" device="-0603-25V-(+80/-20%)" package3d_urn="urn:adsk.eagle:package:37414/1" value="0.1uF"/>
 <part name="SUPPLY3" library="SparkFun-PowerSymbols" library_urn="urn:adsk.eagle:library:530" deviceset="VIN" device="" value="VINR"/>
-<part name="L1" library="inductors" library_urn="urn:adsk.eagle:library:243" deviceset="BLM15H" device="" package3d_urn="urn:adsk.eagle:package:15132/1" technology="B221SN1"/>
+<part name="L1" library="52101-101-REV-A_v16" library_urn="urn:adsk.eagle:library:21899384" deviceset="RC-MASTER-SMD_FB_" device="0805MP" package3d_urn="urn:adsk.eagle:package:15662270/2"/>
 <part name="SUPPLY7" library="SparkFun-PowerSymbols" library_urn="urn:adsk.eagle:library:530" deviceset="3.3V" device=""/>
 <part name="U$1" library="SparkFun-PowerSymbols" library_urn="urn:adsk.eagle:library:530" deviceset="VDDA" device=""/>
@@
 <wire x1="360.68" y1="124.46" x2="360.68" y2="121.92" width="0.1524" layer="91"/>
 <pinref part="L1" gate="G$1" pin="1"/>
-<wire x1="360.68" y1="121.92" x2="363.22" y2="121.92" width="0.1524" layer="91"/>
+<wire x1="360.68" y1="121.92" x2="365.76" y2="121.92" width="0.1524" layer="91"/>
 </segment>
 <segment>
@@
 <pinref part="L1" gate="G$1" pin="2"/>
 <pinref part="VDDA2" gate="G$1" pin="1"/>
-<wire x1="373.38" y1="121.92" x2="378.46" y2="121.92" width="0.1524" layer="91"/>
+<wire x1="370.84" y1="121.92" x2="378.46" y2="121.92" width="0.1524" layer="91"/>
 <wire x1="378.46" y1="121.92" x2="383.54" y2="121.92" width="0.1524" layer="91"/>
 <wire x1="383.54" y1="121.92" x2="388.62" y2="121.92" width="0.1524" layer="91"/>
