File: STM32F102CBT6/Yeni klasör/ATESLEME.sch (EAGLE design)
At the start: 55 parts, among them U1 ADXL345PATRICK, U3 AMS1117-3.3, U4 STM32F102CBT6, Y2 ABM2B-8.000MHZ-10-1-U-T

Commit message: NMOS trace was be expanded and 1206 package version was created
Parts:
- ADXLC1, CRST, LPSC1, LPSC2, OSCC1, OSCC2, RC2, RC3, VBAT, VDD, VDD1, VDD2, VDD3, VDDA1, VDDA2: device SparkFun-Capacitors:0.1UF-0603-25V-(+80/-20%) -> 52101-101-REV-A_v16:RC-MASTER-SMD_C_1206MP
- APGRD, MNRD, S, S2, VBAT_D: value 3.3k -> 3k3; device SparkFun-Resistors:2.0KOHM1/10W5%(0603) -> SparkFun-Resistors:10OHM-1206-1/4W-1%
- APGRU, BOOT0, G1, G2, LED4, MNRU, NRST, VBAT_U: device SparkFun-Resistors:2.0KOHM1/10W5%(0603) -> SparkFun-Resistors:10OHM-1206-1/4W-1%
- BUZ: value 22R -> 22; device SparkFun-Resistors:2.0KOHM1/10W5%(0603) -> SparkFun-Resistors:10OHM-1206-1/4W-1%
- F: device SparkFun-Fuses:PPTC_THREE-QUARTER-AMP -> 52101-101-REV-A_v16:RC-MASTER-SMD_FB_1206MP
- L1: value BLM15HB221SN1 -> (none); device inductors:BLM15HB221SN1 -> 52101-101-REV-A_v16:RC-MASTER-SMD_FB_1206MP
- LED: device SparkFun-LED:LED-RED0603 -> SparkFun-LED:LED1206
- RD: device SparkFun-LED:LED-RED0603-SMART -> SparkFun-LED:LED1206
- RRO: value 1.5k -> 330; device SparkFun-Resistors:2.0KOHM1/10W5%(0603) -> SparkFun-Resistors:10OHM-1206-1/4W-1%
- SCL_3V3, SDA_3V3: value 4.7k -> 4k7; device SparkFun-Resistors:2.0KOHM1/10W5%(0603) -> SparkFun-Resistors:10OHM-1206-1/4W-1%
