File: STM32F102CBT6/REV2.0/ATESLEME.sch (EAGLE design)
At the start: 65 parts, among them U1 ADXL345PATRICK, U2 MS561101BA03-50, U3 AMS1117-3.3, U4 STM32F102CBT6, U5 38kHz, X1 JST-XH-04-PIN-LONG-PAD, Y2 ABM2B-8.000MHZ-10-1-U-T

Commit message: Version 2.0 was updated by brain.dll
Parts:
- added HOLDR, WPR: 10k, SparkFun-Resistors:2.0KOHM1/10W5%(0603)
- added IC1: WS2811-SOP8, adafruit:WS2811-SOP8
Connections:
- removed net PC13: U4A.PC13
- new net CS: IC1.R, U4A.PB12
- new net HOLD: HOLDR.1, IC1.SET, U4A.PA8
- new net MISO: IC1.G, U4A.PB14
- new net MOSI: IC1.DO, U4A.PB15
- new net SCK: IC1.DIN, U4A.PB13
- new net WP: IC1.B, U4A.PC13, WPR.2
- net 3.3V: now also HOLDR.2, IC1.VDD
- net GND: now also IC1.GND, WPR.1
- net LED2: now also U4A.PB4; no longer U4A.PA5
Changed lines of the file:
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@@
 <part name="GND9" library="SparkFun-PowerSymbols" library_urn="urn:adsk.eagle:library:530" deviceset="GND" device=""/>
 <part name="IRR1" library="SparkFun-Resistors" deviceset="2.0KOHM1/10W5%(0603)" device="" value="1.5k"/>
+<part name="IC1" library="adafruit" library_urn="urn:adsk.eagle:library:420" deviceset="WS2811" device="-SOP8" package3d_urn="urn:adsk.eagle:package:6240863/1"/>
+<part name="GND11" library="SparkFun-PowerSymbols" library_urn="urn:adsk.eagle:library:530" deviceset="GND" device=""/>
+<part name="SUPPLY15" library="SparkFun-PowerSymbols" library_urn="urn:adsk.eagle:library:530" deviceset="3.3V" device=""/>
+<part name="HOLDR" library="SparkFun-Resistors" deviceset="2.0KOHM1/10W5%(0603)" device="" value="10k"/>
+<part name="WPR" library="SparkFun-Resistors" deviceset="2.0KOHM1/10W5%(0603)" device="" value="10k"/>
 </parts>
 <sheets>
@@
 <attribute name="VALUE" x="133.858" y="166.37" size="1.778" layer="96" rot="R270"/>
 </instance>
+<instance part="IC1" gate="G$1" x="71.12" y="114.3" smashed="yes">
+<attribute name="NAME" x="63.5" y="106.68" size="1.778" layer="95"/>
+</instance>
+<instance part="GND11" gate="1" x="53.34" y="106.68" smashed="yes">
+<attribute name="VALUE" x="53.34" y="106.426" size="1.778" layer="96" align="top-center"/>
+</instance>
+<instance part="SUPPLY15" gate="G$1" x="88.9" y="121.92" smashed="yes">
+<attribute name="VALUE" x="88.9" y="124.714" size="1.778" layer="96" align="bottom-center"/>
+</instance>
+<instance part="HOLDR" gate="G$1" x="96.52" y="119.38" smashed="yes" rot="R180">
+<attribute name="NAME" x="100.33" y="117.8814" size="1.778" layer="95" rot="R180"/>
+<attribute name="VALUE" x="100.33" y="122.682" size="1.778" layer="96" rot="R180"/>
+</instance>
+<instance part="WPR" gate="G$1" x="45.72" y="111.76" smashed="yes" rot="R180">
+<attribute name="NAME" x="49.53" y="110.2614" size="1.778" layer="95" rot="R180"/>
+<attribute name="VALUE" x="49.53" y="115.062" size="1.778" layer="96" rot="R180"/>
+</instance>
 </instances>
 <busses>
@@
 <wire x1="154.94" y1="137.16" x2="154.94" y2="139.7" width="0.1524" layer="91"/>
 </segment>
+<segment>
+<pinref part="GND11" gate="1" pin="GND"/>
+<pinref part="IC1" gate="G$1" pin="GND"/>
+<wire x1="53.34" y1="109.22" x2="53.34" y2="111.76" width="0.1524" layer="91"/>
+<wire x1="53.34" y1="111.76" x2="58.42" y2="111.76" width="0.1524" layer="91"/>
+<pinref part="WPR" gate="G$1" pin="1"/>
+<wire x1="50.8" y1="111.76" x2="53.34" y2="111.76" width="0.1524" layer="91"/>
+<junction x="53.34" y="111.76"/>
+</segment>
 </net>
 <net name="VCC" class="0">
@@
 <wire x1="154.94" y1="129.54" x2="154.94" y2="127" width="0.1524" layer="91"/>
 </segment>
+<segment>
+<pinref part="SUPPLY15" gate="G$1" pin="3.3V"/>
+<pinref part="IC1" gate="G$1" pin="VDD"/>
+<wire x1="88.9" y1="121.92" x2="88.9" y2="119.38" width="0.1524" layer="91"/>
+<wire x1="88.9" y1="119.38" x2="83.82" y2="119.38" width="0.1524" layer="91"/>
+<pinref part="HOLDR" gate="G$1" pin="2"/>
+<wire x1="91.44" y1="119.38" x2="88.9" y2="119.38" width="0.1524" layer="91"/>
+<junction x="88.9" y="119.38"/>
+</segment>
 </net>
 <net name="N$2" class="0">
@@
 <wire x1="266.7" y1="129.54" x2="271.78" y2="129.54" width="0.1524" layer="91"/>
 <label x="271.78" y="129.54" size="1.27" layer="95" xref="yes"/>
-</segment>
-</net>
-<net name="PC13" class="0">
-<segment>
-<pinref part="U4" gate="A" pin="PC13"/>
-<wire x1="266.7" y1="154.94" x2="271.78" y2="154.94" width="0.1524" layer="91"/>
-<label x="271.78" y="154.94" size="1.27" layer="95" xref="yes"/>
 </segment>
 </net>
@@
 <net name="LED2" class="0">
 <segment>
-<pinref part="U4" gate="A" pin="PA5"/>
-<wire x1="205.74" y1="142.24" x2="200.66" y2="142.24" width="0.1524" layer="91"/>
-<label x="200.66" y="142.24" size="1.27" layer="95" rot="R180" xref="yes"/>
-</segment>
-<segment>
 <pinref part="LED1" gate="G$1" pin="1"/>
 <wire x1="127" y1="190.5" x2="121.92" y2="190.5" width="0.1524" layer="91"/>
 <label x="121.92" y="190.5" size="1.27" layer="95" rot="R180" xref="yes"/>
 </segment>
+<segment>
+<pinref part="U4" gate="A" pin="PB4"/>
+<wire x1="205.74" y1="101.6" x2="200.66" y2="101.6" width="0.1524" layer="91"/>
+<label x="200.66" y="101.6" size="1.27" layer="95" rot="R180" xref="yes"/>
+</segment>
 </net>
 <net name="N$6" class="0">
@@
 </segment>
 </net>
+<net name="CS" class="0">
+<segment>
+<pinref part="IC1" gate="G$1" pin="R"/>
+<wire x1="58.42" y1="119.38" x2="53.34" y2="119.38" width="0.1524" layer="91"/>
+<label x="53.34" y="119.38" size="1.27" layer="95" rot="R180" xref="yes"/>
+</segment>
+<segment>
+<pinref part="U4" gate="A" pin="PB12"/>
+<wire x1="205.74" y1="81.28" x2="200.66" y2="81.28" width="0.1524" layer="91"/>
+<label x="200.66" y="81.28" size="1.27" layer="95" rot="R180" xref="yes"/>
+</segment>
+</net>
+<net name="MISO" class="0">
+<segment>
+<pinref part="IC1" gate="G$1" pin="G"/>
+<wire x1="58.42" y1="116.84" x2="53.34" y2="116.84" width="0.1524" layer="91"/>
+<label x="53.34" y="116.84" size="1.27" layer="95" rot="R180" xref="yes"/>
+</segment>
+<segment>
+<pinref part="U4" gate="A" pin="PB14"/>
+<wire x1="205.74" y1="76.2" x2="200.66" y2="76.2" width="0.1524" layer="91"/>
+<label x="200.66" y="76.2" size="1.27" layer="95" rot="R180" xref="yes"/>
+</segment>
+</net>
+<net name="WP" class="0">
+<segment>
+<pinref part="IC1" gate="G$1" pin="B"/>
+<wire x1="58.42" y1="114.3" x2="40.64" y2="114.3" width="0.1524" layer="91"/>
+<label x="38.1" y="114.3" size="1.27" layer="95" rot="R180" xref="yes"/>
+<pinref part="WPR" gate="G$1" pin="2"/>
+<wire x1="40.64" y1="114.3" x2="38.1" y2="114.3" width="0.1524" layer="91"/>
+<wire x1="40.64" y1="111.76" x2="40.64" y2="114.3" width="0.1524" layer="91"/>
+<junction x="40.64" y="114.3"/>
+</segment>
+<segment>
+<pinref part="U4" gate="A" pin="PC13"/>
+<wire x1="266.7" y1="154.94" x2="271.78" y2="154.94" width="0.1524" layer="91"/>
+<label x="271.78" y="154.94" size="1.27" layer="95" xref="yes"/>
+</segment>
+</net>
+<net name="MOSI" class="0">
+<segment>
+<pinref part="IC1" gate="G$1" pin="DO"/>
+<wire x1="83.82" y1="111.76" x2="88.9" y2="111.76" width="0.1524" layer="91"/>
+<label x="88.9" y="111.76" size="1.27" layer="95" xref="yes"/>
+</segment>
+<segment>
+<pinref part="U4" gate="A" pin="PB15"/>
+<wire x1="205.74" y1="73.66" x2="200.66" y2="73.66" width="0.1524" layer="91"/>
+<label x="200.66" y="73.66" size="1.27" layer="95" rot="R180" xref="yes"/>
+</segment>
+</net>
+<net name="SCK" class="0">
+<segment>
+<pinref part="IC1" gate="G$1" pin="DIN"/>
+<wire x1="83.82" y1="114.3" x2="88.9" y2="114.3" width="0.1524" layer="91"/>
+<label x="88.9" y="114.3" size="1.27" layer="95" xref="yes"/>
+</segment>
+<segment>
+<pinref part="U4" gate="A" pin="PB13"/>
+<wire x1="205.74" y1="78.74" x2="200.66" y2="78.74" width="0.1524" layer="91"/>
+<label x="200.66" y="78.74" size="1.27" layer="95" rot="R180" xref="yes"/>
+</segment>
+</net>
+<net name="HOLD" class="0">
+<segment>
+<pinref part="IC1" gate="G$1" pin="SET"/>
+<wire x1="83.82" y1="116.84" x2="104.14" y2="116.84" width="0.1524" layer="91"/>
+<label x="106.68" y="116.84" size="1.27" layer="95" xref="yes"/>
+<pinref part="HOLDR" gate="G$1" pin="1"/>
+<wire x1="104.14" y1="116.84" x2="106.68" y2="116.84" width="0.1524" layer="91"/>
+<wire x1="101.6" y1="119.38" x2="104.14" y2="119.38" width="0.1524" layer="91"/>
+<wire x1="104.14" y1="119.38" x2="104.14" y2="116.84" width="0.1524" layer="91"/>
+<junction x="104.14" y="116.84"/>
+</segment>
+<segment>
+<pinref part="U4" gate="A" pin="PA8"/>
+<wire x1="205.74" y1="134.62" x2="200.66" y2="134.62" width="0.1524" layer="91"/>
+<label x="200.66" y="134.62" size="1.27" layer="95" rot="R180" xref="yes"/>
+</segment>
+</net>

Commit message: VDDA cap calue was changed
Parts:
- IC1: value WS2811-SOP8 -> EN25F40-100GCP-TR
- S, S2: value 3.3k -> 4.7k
- U8, U9: value (none) -> SI2308CDS-T1-GE3
- VDDA2: value 100nF -> 10nF
Other:
- note removed: "MCU"
