File: STM32F102CBT6/REV3.0/ATESLEME.sch (EAGLE design)
At the start: 68 parts, among them IC1 EN25F40-100GCP-TR, U1 ADXL345PATRICK, U2 MS561101BA03-50, U3 AMS1117-3.3, U4 STM32F102CBT6, U5 38kHz, U8 SI2308CDS-T1-GE3, U9 SI2308CDS-T1-GE3, X1 JST-XH-04-PIN-LONG-PAD, Y2 ABM2B-8.000MHZ-10-1-U-T

Commit message: Regulator was added for e match and released new two version for ordering
Parts:
- removed APGLED, MNLED, S, S2: 4.7k, SparkFun-Resistors:2.0KOHM1/10W5%(0603)
- removed APGRD, MNRD: 3.3k, SparkFun-Resistors:2.0KOHM1/10W5%(0603)
- removed APGRU, MNRU: 10k, SparkFun-Resistors:2.0KOHM1/10W5%(0603)
- removed ESDA, ESDM: 12V, Wurth_EMC Components_WE-TVSP:WE-TVSP_DO-214AC_400W_UNI_824500102
- removed G1, G2: 22, SparkFun-Resistors:2.0KOHM1/10W5%(0603)
- removed RD1, RD2: Blue, SparkFun-LED:LED-RED0603-SMART
- removed U8, U9: SI2308CDS-T1-GE3, IRLML6344TRPBF:IRLML6344TRPBF
- added APGLED1, MNLED1, S1, S3: 4.7k, SparkFun-Resistors:2.0KOHM1/10W5%(0603)
- added APGRD1, MNRD1: 3.3k, SparkFun-Resistors:2.0KOHM1/10W5%(0603)
- added APGRU1, MNRU1: 10k, SparkFun-Resistors:2.0KOHM1/10W5%(0603)
- added C2, C6: 22uF, SparkFun-Capacitors:47UF-POLAR-EIA3528-10V-10%
- added C3, C4: 100nF, SparkFun-Capacitors:1.0UF-0603-16V-10%
- added D2: B5819W, Diode:SCHOTTKY_MBR0520LT1GDO-219
- added D9: (no value), SparkFun-LED:LED0603
- added ESDA1, ESDM1: 12V, Wurth_EMC Components_WE-TVSP:WE-TVSP_DO-214AC_400W_UNI_824500102
- added G3, G4: 22, SparkFun-Resistors:2.0KOHM1/10W5%(0603)
- added Q1: STS4DNF60L, STS4DNF60L:STS4DNF60L
- added R17: 1k5, SparkFun-Resistors:1KOHM-0603-1/10W-1%
- added RD3, RD4: Blue, SparkFun-LED:LED-RED0603-SMART
- added U7: AMS1117-3.3, AMS1117-3.3:AMS1117-3.3
Connections:
- removed net N$14: ESDA.C, G1.1, S.1, U8.G
- removed net N$3 (its old number): MNLED.1, RD1.A
- new net 5V: APOGEE.1, C4.1, C6.+, MAIN.2, R17.2, U7.VOUT
- new net HT1: U7.HT
- new net N$11: ESDA1.C, G4.1, Q1.G2, S3.2
- new net N$12: APGLED1.1, RD4.A
- new net N$7: ESDM1.C, G3.1, Q1.G1, S1.2
- new net N$9: MNLED1.1, RD3.A
- net APG: now also G4.2, U4A.PB3; no longer G1.2, U4A.PA15
- net GND: now also APGRD1.1, C2.-, C3.2, C4.2, C6.-, D9.C, ESDA1.A, ESDM1.A, MNRD1.1, Q1.S1, Q1.S2, RD3.C, RD4.C, S1.1, S3.1, U7.ADJ; no longer APGRD.1, ESDA.A, ESDM.A, MNRD.1, RD1.C, RD2.C, S.2, S2.2, U8.S, U9.S
- net MN: now also G3.2, U4A.PA15; no longer G2.2, U4A.PB3
- net N$4: now also C2.+, C3.1, D2.C, U7.VIN; no longer APGLED.1, RD2.A
- net N$8: now also D9.A, R17.1; no longer ESDM.C, G2.1, S2.1, U9.G
- net VAPG: now also APGLED1.2, APGRU1.2, APOGEE.2, Q1.D2; no longer APGLED.2, APGRU.2, APOGEE.1, U8.D
- net VAPGS: now also APGRD1.2, APGRU1.1, U4A.PA7; no longer APGRD.2, APGRU.1, U4A.PB0
- net VIN: now also D2.A; no longer APOGEE.2, MAIN.2
- net VMN: now also MNLED1.2, MNRU1.2, Q1.D1; no longer MNLED.2, MNRU.2, U9.D
- net VMNS: now also MNRD1.2, MNRU1.1, U4A.PB0; no longer MNRD.2, MNRU.1, U4A.PA7
Other:
- note added: "GÜÇ DEVRELERİ"
- note removed: "APOGEE"
- note removed: "MAIN"

Commit message: Sotware and Algorithm was added
Parts:
- U7: value AMS1117-3.3 -> AMS1117-5.0
Changed lines of the file:
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@@
 <part name="D2" library="Diode" library_urn="urn:adsk.eagle:library:16378169" deviceset="SCHOTTKY_" device="DO-219" package3d_urn="urn:adsk.eagle:package:9427153/2" technology="MBR0520LT1G" value="B5819W"/>
 <part name="SUPPLY16" library="SparkFun-PowerSymbols" library_urn="urn:adsk.eagle:library:530" deviceset="5V" device=""/>
-<part name="U7" library="AMS1117-3.3" library_urn="urn:adsk.eagle:library:27162810" deviceset="AMS1117-3.3" device="" package3d_urn="urn:adsk.eagle:package:27162813/2"/>
+<part name="U7" library="AMS1117-3.3" library_urn="urn:adsk.eagle:library:27162810" deviceset="AMS1117-3.3" device="" package3d_urn="urn:adsk.eagle:package:27162813/2" value="AMS1117-5.0"/>
 <part name="GND36" library="supply1" library_urn="urn:adsk.eagle:library:371" deviceset="GND" device=""/>
 <part name="D9" library="SparkFun-LED" library_urn="urn:adsk.eagle:library:27167846" deviceset="LED" device="0603" package3d_urn="urn:adsk.eagle:package:27167834/2"/>
